File: PMS/PCB/ADC.kicad_sch (KiCad schematic)
At the start: 9 parts

Commit message: Correcciones menores
mentirillas
Parts:
- gave numbers to parts that had none: 9
Other:
- company: (none) -> Misión LAMBDA
- title: (none) -> PMS - Monitoreo de Reguladores
- moved on the sheet: C501, C502, F501, F502, R501, R502, R503, R504, U501
