File: PMS/PCB/Regulador_12V.kicad_sch (KiCad schematic)
At the start: 16 parts, among them U7 MP1584

Commit message: Correcciones menores
mentirillas
Parts:
- removed R4: R, symbol Device:R
- renumbered C4 to C201, C6 to C202, C1 to C203, C2 to C204, C5 to C205, C3 to C206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
Connections:
- net V_In renamed VSYS
Other:
- company: (none) -> Misión LAMBDA
- title: (none) -> PMS - Regulador 12V
