File: PMS/PCB/PMS.kicad_sch (KiCad schematic)
At the start: 0 parts

Commit message: Define ciertos pines y diseña mediciones
Parts:
- added C13, C15: 22u, symbol Device:C
- added C14, C16: 0.1u, symbol Device:C
- added C17: 100n, symbol Device:C
- added D1: SS24, Diode_SMD:D_SMA, symbol Diode:SS24
- added D4: LED, symbol Device:LED
- added Q1: PMOS, symbol Simulation_SPICE:PMOS
- added R1, R2, R3: R, symbol Device:R
- added R12: 1000, symbol Device:R
- added R13, R15: 1M, symbol Device:R
- added R14: 620k, symbol Device:R
- added R16: 10M, symbol Device:R
- added U2, U3: LM2904, symbol Amplifier_Operational:LM2904
- added U5: LM1117MP-ADJ, Package_TO_SOT_SMD:SOT-223-3_TabPin2, symbol Regulator_Linear:LM1117MP-ADJ
- added U6: ATmega328P-A, Package_QFP:TQFP-32_7x7mm_P0.8mm, symbol MCU_Microchip_ATmega:ATmega328P-A
Connections:
- new net: Q1.2 (G), U3.1
- new net: R1.1, R2.2, U3.2 (-)
- new net: C17.2, U6.4 (VCC), U6.6 (VCC)
- new net: D4.1 (K), R12.1
- new net +12V: R13.1
- new net +3V3: C13.1, C14.1, D4.2 (A), U5.2 (VO), U6.25 (PC2)
- new net +5V: C15.1, C16.1, C17.1, R15.1, U5.3 (VI)
- new net EN_12V: U6.13 (PB1)
- new net EN_5V: U6.12 (PB0)
- new net GND: C13.2, C14.2, C15.2, C16.2, R1.2, R12.2, R14.2, R16.2, R3.2, U2.4 (V-), U5.1 (ADJ), U6.21 (GND), U6.3 (GND), U6.5 (GND)
- new net PWM1: U6.1 (PD3)
- new net PWM2: U6.9 (PD5)
- new net PWM3: U6.14 (PB2)
- new net RX: U6.30 (PD0)
- new net SCL: U6.28 (PC5)
- new net SDA: U6.27 (PC4)
- new net TX: U6.31 (PD1)
- new net V_12V: R13.2, R14.1, U6.23 (PC0)
- new net V_5V: R15.2, R16.1, U6.24 (PC1)
- new net V_Bat: Q1.3 (S), R2.1, U2.8 (V+)
- new net V_Ext: D1.2 (A), R3.1, U3.3 (+)
- new net V_In: D1.1 (K), Q1.1 (D)
Other:
- added sheet Regulador 12 V (Regulador_12V.kicad_sch)
- added sheet Regulador 5 V (Regulador_5V.kicad_sch)

Commit message: Continua Desarrollo
Parts:
- removed C13, C15: 22u, symbol Device:C
- removed C14, C16: 0.1u, symbol Device:C
- removed D4: LED, symbol Device:LED
- removed R12: 1000, symbol Device:R
- removed U5: LM1117MP-ADJ, Package_TO_SOT_SMD:SOT-223-3_TabPin2, symbol Regulator_Linear:LM1117MP-ADJ
- added F4: Polyfuse, symbol Device:Polyfuse
- added J1: PMS-OBC, symbol Connector_Generic:Conn_01x06
- added J2: PMS-TRU, symbol Connector_Generic:Conn_01x06
- added J3: PMS-BAT_CELLS, symbol Connector_Generic:Conn_01x06
- added J4: PMS-PROG, symbol Connector_Generic:Conn_01x04
- added J5: PMS-BAT_TEMP, symbol Connector_Generic:Conn_01x02
- added J6: BAT_IN, symbol Connector_Generic:Conn_01x02
- added R23: 1M, symbol Device:R
- added R24: 10M, symbol Device:R
- R1: value R -> 4K7
- R2: value R -> 1K
- R3: value R -> 10K
Connections:
- net +3V3: now also J1.4 (Pin_4), R23.1
- net +5V: now also J1.5 (Pin_5), J4.4 (Pin_4), J5.1 (Pin_1)
- net GND: now also J1.3 (Pin_3), J1.6 (Pin_6), J3.1 (Pin_1), J4.1 (Pin_1), J6.1 (Pin_1), R24.2
- net RX: now also J4.2 (Pin_2)
- net SCL: now also J1.2 (Pin_2)
- net SDA: now also J1.1 (Pin_1)
- net TX: now also J4.3 (Pin_3)
- net V_12V: no longer U6.23 (PC0)
- net V_5V: no longer U6.24 (PC1)
- net V_Bat renamed +BATT
- net +BATT: now also F4.1
- new net: F4.2, J6.2 (Pin_2)
- new net BAT_TEMP: J5.2 (Pin_2)
- new net PELT1_A: J2.1 (Pin_1)
- new net PELT1_B: J2.2 (Pin_2)
- new net PELT2_A: J2.3 (Pin_3)
- new net PELT2_B: J2.4 (Pin_4)
- new net PELT3_A: J2.5 (Pin_5)
- new net PELT3_B: J2.6 (Pin_6)
- new net VBAT1: J3.2 (Pin_2)
- new net VBAT2: J3.3 (Pin_3)
- new net VBAT3: J3.4 (Pin_4)
- new net VBAT4: J3.5 (Pin_5)
- new net VBAT5: J3.6 (Pin_6)
- new net V_3V3: R23.2, R24.1
Other:
- added sheet ADC (ADC.kicad_sch)
- added sheet Regulador 3.3V (Regulador_3.3V.kicad_sch)
- sheet Regulador 12 V ports: added EN; removed ENBLE
- sheet Regulador 5 V ports: added EN; removed ENBLE
- moved on the sheet: D1, R1, R13, R14, R15, R16, R2

Commit message: Diseña sensor de corriente y puentes H
Parts:
- removed R24: 10M, symbol Device:R
- added C20, C21, C22, C23, C24, C27: 100n, symbol Device:C
- added C25: 4.7u, symbol Device:C
- added C26: 1u, symbol Device:C
- added C28: 1n, symbol Device:C
- added SW1: SW_Push, symbol Switch:SW_Push
- added U5, U8: L298HN, Package_TO_SOT_THT:TO-220-15_P2.54x2.54mm_StaggerOdd_Lead5.84mm_TabDown, symbol Driver_Motor:L298HN
- added U9: ACS712xLCTR-30A, Package_SO:SOIC-8_3.9x4.9mm_P1.27mm, symbol Sensor_Current:ACS712xLCTR-30A
- added Y2: 16 MHz, symbol Device:Crystal_GND2
- C17: value 100n -> 1u
- R23: value 1M -> 1k
Connections:
- net V_3V3 is gone; now on an unnamed net: R23.2
- net +12V: now also C21.1, C23.1, U5.4 (Vs), U8.4 (Vs)
- net +3V3: no longer R23.1, U6.25 (PC2)
- net +5V: now also C17.2, R23.1, U6.18 (AVCC), U6.4 (VCC), U6.6 (VCC), C20.2, C22.2, C25.2, C26.2, C27.2, U5.9 (Vss), U8.9 (Vss), U9.8 (VCC); no longer C17.1
- net GND: now also C17.1, C20.1, C21.2, C22.1, C23.2, C24.1, C25.1, C26.1, C27.1, SW1.2, U5.8 (GND), U8.10 (IN3), U8.11 (EnB), U8.12 (IN4), U8.8 (GND), Y2.2
- net PELT1_A: now also U5.2 (OUT1)
- net PELT1_B: now also U5.3 (OUT2)
- net PELT2_A: now also U5.13 (OUT3)
- net PELT2_B: now also U5.14 (OUT4)
- net PELT3_A: now also U8.2 (OUT1)
- net PELT3_B: now also U8.3 (OUT2)
- net PWM1: now also U5.6 (EnA)
- net PWM2: now also U5.11 (EnB)
- net PWM3: now also U8.6 (EnA)
- net VBAT1: now also U6.23 (PC0)
- net VBAT2: now also U6.24 (PC1)
- net VBAT3: now also U6.25 (PC2)
- net VBAT4: now also U6.19 (ADC6)
- net VBAT5: now also U6.22 (ADC7)
- net V_In: now also U9.1 (IP+), U9.2 (IP+)
- net SDA_Soft: now reaches U6.10 (PD6)
- net SCL_Soft: now reaches U6.11 (PD7)
- net PELT1_CTRL_1: now reaches U6.15 (PB3)
- net PELT1_CTRL_1: now also U5.5 (IN1)
- net PELT1_CTRL_2: now reaches U6.16 (PB4)
- net PELT1_CTRL_2: now also U5.7 (IN2)
- net PELT2_CTRL_1: now reaches U6.17 (PB5)
- net PELT2_CTRL_1: now also U5.10 (IN3)
- net at U6.20 (AREF): now also C24.2
- net Corriente: now reaches U6.26 (PC3)
- net Corriente: now also U9.7 (VIOUT)
- net at U6.29 (~{RESET}/PC6): now also SW1.1
- net PELT2_CTRL_2: now reaches U6.32 (PD2)
- net PELT2_CTRL_2: now also U5.12 (IN4)
- net at U6.7 (XTAL1/PB6): now also Y2.3
- net at U6.8 (XTAL2/PB7): now also Y2.1
- new net: C28.1, U9.5 (GND)
- new net: C28.2, U9.6 (FILTER)
- new net PELT3_CTRL_1: U8.5 (IN1)
- new net PELT3_CTRL_2: U8.7 (IN2)
- new net V_Sys: U9.3 (IP-), U9.4 (IP-)
Other:
- moved on the sheet: C17, U6

Commit message: Cambia sensor de corriente
Parts:
- removed C28: 1n, symbol Device:C
- removed U9: ACS712xLCTR-30A, Package_SO:SOIC-8_3.9x4.9mm_P1.27mm, symbol Sensor_Current:ACS712xLCTR-30A
- added R24, R25: 10k, symbol Device:R
- added R26: R, symbol Device:R
- added U10: INA219AxDCN, Package_TO_SOT_SMD:SOT-23-8, symbol Sensor_Energy:INA219AxDCN
Connections:
- net +5V: now also R24.1, R25.1, U10.4 (VS)
- net GND: now also U10.3 (GND), U10.7 (A0), U10.8 (A1)
- net SCL_Soft: now also R25.2, U10.5 (SCL)
- net SDA_Soft: now also R24.2, U10.6 (SDA)
- net V_In: now also R26.1, U10.1 (IN+)
- net V_Sys: now also R26.2, U10.2 (IN-)

Commit message: Correcciones menores
mentirillas
Parts:
- removed C17: 1u, symbol Device:C
- removed C20, C21, C22, C23, C27: 100n, symbol Device:C
- removed D1: SS24, Diode_SMD:D_SMA, symbol Diode:SS24
- removed Q1: PMOS, symbol Simulation_SPICE:PMOS
- removed R1: 4K7, symbol Device:R
- removed R13, R15: 1M, symbol Device:R
- removed R14: 620k, symbol Device:R
- removed R16: 10M, symbol Device:R
- removed R2: 1K, symbol Device:R
- removed R3: 10K, symbol Device:R
- removed U2, U3: LM2904, symbol Amplifier_Operational:LM2904
- removed U5, U8: L298HN, Package_TO_SOT_THT:TO-220-15_P2.54x2.54mm_StaggerOdd_Lead5.84mm_TabDown, symbol Driver_Motor:L298HN
- added C103: 1u, symbol Device:C
- added C105: 100n, symbol Device:C
- added F102: Polyfuse, symbol Device:Polyfuse
- added J104: EXT_IN, symbol Connector_Generic:Conn_01x02
- added R103: 4K7, symbol Device:R
- renumbered C26 to C101, C25 to C102, C24 to C104, F4 to F101, J6 to J101, J2 to J102, J4 to J103, J3 to J105, J1 to J106, J5 to J107, R24 to R101, R25 to R102, R23 to R104, R26 to R105, SW1 to SW101, U6 to U101, U10 to U102, Y2 to Y101
Connections:
- net PELT1_CTRL_1 is gone; now on net PWM3: U101.15 (PB3)
- net PELT2_CTRL_2 is gone; now on net EN_3V3: U101.32 (PD2)
- net +5V: now also C105.1; no longer C101.2, C102.2, R104.1, U101.18 (AVCC), U101.4 (VCC), U101.6 (VCC)
- net BAT_TEMP: now also U101.22 (ADC7), R103.1
- net EN_12V: now also U101.2 (PD4); no longer U101.13 (PB1)
- net EN_5V: now also U101.1 (PD3); no longer U101.12 (PB0)
- net GND: now also C101.2, C102.2, C104.2, C103.2, C105.2, J104.1 (Pin_1), R103.2; no longer C101.1, C102.1, C104.1
- net PWM1: now also U101.13 (PB1); no longer U101.1 (PD3)
- net PWM2: now also U101.14 (PB2); no longer U101.9 (PD5)
- net PWM3: no longer U101.14 (PB2)
- net VBAT2: no longer U101.24 (PC1)
- net VBAT3: no longer U101.25 (PC2)
- net VBAT4: no longer U101.19 (ADC6)
- net VBAT5: no longer U101.22 (ADC7)
- net at U101.20 (AREF): now also C104.1; no longer C104.2
- net Corriente renamed V_VBAT4
- net PELT1_CTRL_2 renamed PELT2_MODE
- net PELT2_CTRL_1 renamed PELT3_MODE
- net V_Sys renamed VSYS
- new net: F102.2, J104.2 (Pin_2)
- new net +5V_SB: C101.1, C102.1, C103.1, R104.1, U101.18 (AVCC), U101.4 (VCC), U101.6 (VCC)
- new net +VEXT: F102.1
- new net CUBESAT_EN: U101.9 (PD5)
- new net PELT1_MODE: U101.12 (PB0)
- new net V_VBAT2: U101.24 (PC1)
- new net V_VBAT3: U101.25 (PC2)
- new net V_VBAT5: U101.19 (ADC6)
- no-connect marks 0 -> 3
Other:
- added sheet Acc. señales (acc_senales.kicad_sch)
- added sheet Control Fuente (control_fuente.kicad_sch)
- added sheet Llaves H (llaves_h.kicad_sch)
- sheet Regulador 12 V ports: added none; removed V_In
- sheet Regulador 3.3V ports: added none; removed V_In
- sheet Regulador 5 V ports: added V_Out_SB; removed V_In
- note added: "Accondicionamiento de Señales"
- note added: "Conectores"
- note added: "Controlador PMS"
- note added: "Controlador Peltier"
- note added: "Entrada de Alimentacion"
- note added: "Monitoreo de Reguladores"
- note added: "Reguladores de voltaje"
- note added: "Sensor de Corriente"
- company: (none) -> Misión LAMBDA
- title: (none) -> Sistema de Administración de Energía (PMS)
- moved on the sheet: C101, C102, C104, F101, J101, J102, J103, J105, J106, J107, R101, R102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

Commit message: Agrega HMI y expansor I2C
Parts:
- added J108: HMI, symbol Connector_Generic:Conn_01x06
Connections:
- net GND: now also J108.2 (Pin_2), J108.4 (Pin_4), J108.6 (Pin_6)
- net PELT1_MODE: no longer U101.12 (PB0)
- net PELT2_MODE: no longer U101.16 (PB4)
- net PELT3_MODE: no longer U101.17 (PB5)
- net SCL_Soft: now also U101.17 (PB5); no longer U101.11 (PD7)
- net SDA_Soft: now also U101.16 (PB4); no longer U101.10 (PD6)
- net CUBESAT_EN renamed HMI_A0
- net HMI_A0: now also J108.5 (Pin_5)
- new net HMI_A1: J108.3 (Pin_3), U101.10 (PD6)
- new net HMI_A2: J108.1 (Pin_1), U101.11 (PD7)
- no-connect marks 3 -> 5
Other:
- added sheet Expansor I2C a Paralelo (expansor_i2c.kicad_sch)
- sheet Control Fuente ports: added none; removed ~{EN}
- note added: "Conector HMI"
- note added: "Expansor I2C"
