File: PMS/PCB/control_fuente.kicad_sch (KiCad schematic)
At the start: 10 parts, among them Q801 IRF9630, Q802 IRF9630, U801 LM2904

Commit message: Agrega HMI y expansor I2C
Parts:
- removed Q801: IRF9630, symbol Simulation_SPICE:PMOS
- removed R801: 100K, symbol Device:R
- removed R803: 18K, symbol Device:R
- removed R804: 10K, symbol Device:R
- removed unit 2 of U801
- renumbered Q802 to Q801, R802 to R801, R805 to R802, R806 to R803
Connections:
- net +VO: now also D801.1 (K), Q801.1 (D)
